File: schematic/doorbell.kicad_sch (KiCad schematic)
At the start: 12 parts, among them J1 door button, P1 Conn_01x02_Socket, SW1 door button, SW2 test

Commit message: ajout résistance R3
Parts:
- added R3: 10K, symbol Device:R
Connections:
- net Vdd: now also R3.1
- net at U1.1 (PA0/SWIM): now also R3.2
Changed lines of the file:
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@@
 	(paper "A4")
+	(junction
+		(at 195.58 128.27)
+		(diameter 0)
+		(color 0 0 0 0)
+	)
 	(junction
 		(at 194.31 152.4)
@@
 	(wire
 		(pts
-			(xy 180.34 128.27) (xy 208.28 128.27)
+			(xy 180.34 128.27) (xy 195.58 128.27)
 		)
 		(stroke
@@
 	(wire
 		(pts
+			(xy 195.58 135.89) (xy 195.58 144.78)
+		)
+		(stroke
+			(width 0)
+			(type default)
+		)
+	)
+	(wire
+		(pts
 			(xy 226.06 128.27) (xy 226.06 135.89)
 		)
@@
 		(pts
 			(xy 234.95 152.4) (xy 238.76 152.4)
+		)
+		(stroke
+			(width 0)
+			(type default)
+		)
+	)
+	(wire
+		(pts
+			(xy 195.58 128.27) (xy 208.28 128.27)
 		)
 		(stroke
@@
 					(unit 1)
 				)
+			)
+		)
+	)
+	(symbol
+		(lib_id "Device:R")
+		(at 195.58 132.08 0)
+		(unit 1)
+		(exclude_from_sim no)
+		(in_bom yes)
+		(on_board yes)
+		(dnp no)
+		(property "Reference" "R3"
+			(at 197.104 130.81 0)
+			(effects
+				(font
+					(size 1.27 1.27)
+				)
+				(justify left)
+			)
+		)
+		(property "Value" "10K"
+			(at 196.85 133.604 0)
+			(effects
+				(font
+					(size 1.27 1.27)
+				)
+				(justify left)
+			)
+		)
+		(property "Footprint" ""
+			(at 193.802 132.08 90)
+			(effects
+				(font
+					(size 1.27 1.27)
+				)
+				(hide yes)
+			)
+		)
+		(property "Datasheet" "~"
+			(at 195.58 132.08 0)
+			(effects
+				(font
+					(size 1.27 1.27)
+				)
+				(hide yes)
+			)
+		)
+		(property "Description" "Resistor"
+			(at 195.58 132.08 0)
+			(effects
+				(font
+					(size 1.27 1.27)
+				)
+				(hide yes)
+			)
+		)
+		(pin "1"
+		)
+		(pin "2"
+		)
+		(instances
+			(project "doorbell"
+				(path "/446a5a63-b234-4c89-aadd-313415f72588"
+					(reference "R3")
+					(unit 1)
+				)

Commit message: Remplacé condensateur 10µF/16v par 470µF/16v
Parts:
- C3: value 10µF/16V -> 470µF/16V
Changed lines of the file:
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@@
 			)
 		)
-		(property "Value" "10µF/16V"
+		(property "Value" "470µF/16V"
 			(at 231.394 148.844 90)
 			(effects

Commit message: version 2 modification du circuit et du firmware pour ajouter un effet trémolo.
Other:
- added sheet version_2 (version_2.kicad_sch)
- note added: "version 1"
Changed lines of the file:
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@@
+		)
+	)
+	(text "version 1"
+		(exclude_from_sim no)
+		(at 199.644 177.546 0)
+		(effects
+			(font
+				(size 2.54 2.54)
+			)
 		)
 	)
@@
 				)
 			)
+		)
+	)
+	(sheet
+		(at 261.62 163.83)
+		(size 34.29 15.24)
+		(fields_autoplaced yes)
+		(stroke
+			(width 0.1524)
+			(type solid)
+		)
+		(fill
+			(color 0 0 0 0.0000)
+		)
+		(property "Sheetname" "version_2"
+			(at 261.62 163.1184 0)
+			(effects
+				(font
+					(size 1.27 1.27)
+				)
+				(justify left bottom)
+			)
+		)
+		(property "Sheetfile" "version_2.kicad_sch"
+			(at 261.62 179.6546 0)
+			(effects
+				(font
+					(size 1.27 1.27)
+				)
+				(justify left top)
+			)
+		)
+		(instances
+			(project "doorbell"
+				(path "/446a5a63-b234-4c89-aadd-313415f72588"
+					(page "2")
+				)
+			)

Commit message: Ajout du condensateur C6 dans la schématique tag V1.2
Parts:
- added C6: 47nF, symbol Device:C
Connections:
- net GND: now also C6.1
- net at J1.2 (Pin_2), R1.2, SW2.1 (A)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: now also C6.2
Other:
- note added: "version 1.2"
- note removed: "version 1"
Changed lines of the file:
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@@
+	)
+	(junction
+		(at 226.06 128.27)
+		(diameter 0)
+		(color 0 0 0 0)
 	)
 	(junction
@@
 	(wire
 		(pts
+			(xy 226.06 124.46) (xy 226.06 128.27)
+		)
+		(stroke
+			(width 0)
+			(type default)
+		)
+	)
+	(wire
+		(pts
 			(xy 180.34 128.27) (xy 195.58 128.27)
 		)
@@
 		(pts
 			(xy 180.34 149.86) (xy 195.58 149.86)
+		)
+		(stroke
+			(width 0)
+			(type default)
+		)
+	)
+	(wire
+		(pts
+			(xy 224.79 124.46) (xy 226.06 124.46)
 		)
 		(stroke
@@
 		)
 	)
-	(text "version 1"
+	(text "version 1.2"
 		(exclude_from_sim no)
 		(at 199.644 177.546 0)
@@
 	(symbol
 		(lib_id "power:GND")
+		(at 217.17 124.46 270)
+		(unit 1)
+		(exclude_from_sim no)
+		(in_bom yes)
+		(on_board yes)
+		(dnp no)
+		(property "Reference" "#PWR016"
+			(at 210.82 124.46 0)
+			(effects
+				(font
+					(size 1.27 1.27)
+				)
+				(hide yes)
+			)
+		)
+		(property "Value" "GND"
+			(at 212.09 124.46 90)
+			(effects
+				(font
+					(size 1.27 1.27)
+				)
+			)
+		)
+		(property "Footprint" ""
+			(at 217.17 124.46 0)
+			(effects
+				(font
+					(size 1.27 1.27)
+				)
+				(hide yes)
+			)
+		)
+		(property "Datasheet" ""
+			(at 217.17 124.46 0)
+			(effects
+				(font
+					(size 1.27 1.27)
+				)
+				(hide yes)
+			)
+		)
+		(property "Description" "Power symbol creates a global label with name \"GND\" , ground"
+			(at 217.17 124.46 0)
+			(effects
+				(font
+					(size 1.27 1.27)
+				)
+				(hide yes)
+			)
+		)
+		(pin "1"
+		)
+		(instances
+			(project "doorbell"
+				(path "/446a5a63-b234-4c89-aadd-313415f72588"
+					(reference "#PWR016")
+					(unit 1)
+				)
+			)
+		)
+	)
+	(symbol
+		(lib_id "power:GND")
 		(at 219.71 154.94 0)
 		(unit 1)
@@
 	)
 	(symbol
+		(lib_id "Device:C")
+		(at 220.98 124.46 90)
+		(unit 1)
+		(exclude_from_sim no)
+		(in_bom yes)
+		(on_board yes)
+		(dnp no)
+		(property "Reference" "C6"
+			(at 220.98 121.158 90)
+			(effects
+				(font
+					(size 1.27 1.27)
+				)
+			)
+		)
+		(property "Value" "47nF"
+			(at 224.536 122.936 90)
+			(effects
+				(font
+					(size 1.27 1.27)
+				)
+			)
+		)
+		(property "Footprint" ""
+			(at 224.79 123.4948 0)
+			(effects
+				(font
+					(size 1.27 1.27)
+				)
+				(hide yes)
+			)
+		)
+		(property "Datasheet" "~"
+			(at 220.98 124.46 0)
+			(effects
+				(font
+					(size 1.27 1.27)
+				)
+				(hide yes)
+			)
+		)
+		(property "Description" "Unpolarized capacitor"
+			(at 220.98 124.46 0)
+			(effects
+				(font
+					(size 1.27 1.27)
+				)
+				(hide yes)
+			)
+		)
+		(pin "2"
+		)
+		(pin "1"
+		)
+		(instances
+			(project ""
+				(path "/446a5a63-b234-4c89-aadd-313415f72588"
+					(reference "C6")
+					(unit 1)
+				)
+			)
+		)
+	)
+	(symbol
 		(lib_id "Device:LED")
 		(at 219.71 143.51 90)
@@
 	)
 	(sheet
-		(at 261.62 163.83)
-		(size 34.29 15.24)
-		(fields_autoplaced yes)
+		(at 261.62 172.72)
+		(size 19.05 11.43)
 		(stroke
 			(width 0.1524)
@@
 		)
 		(property "Sheetname" "version_2"
-			(at 261.62 163.1184 0)
+			(at 261.62 172.0084 0)
 			(effects
 				(font
@@
 		)
 		(property "Sheetfile" "version_2.kicad_sch"
-			(at 261.62 179.6546 0)
-			(effects
-				(font
+			(at 255.778 184.658 0)
+			(effects
+				(font
